File: kicad/nahs-HeatBrick_v1.0_r1/nahs-HeatBrick_v1.0_r1.kicad_pcb (KiCad board)
At the start: 2 copper layers, 45 x 70 mm, 62 parts, among them IC1 ESP12S, IC2 ATTINY414, J2 AKL 101-02, J3 AKL 101-02, Q1 BSS138, Q3 BS170, SW1 KMR_231_G_LFS, SW2 SSSS820101, SW3 SW_DIP_x04, SW4 Taster_3301, SW5 Taster_4545, U1 MCP1700-3302, U2 LM1086_IT5,0

Commit message: v1.0 R1 ibom done
Parts:
- LED2: value Green -> Red
- moved FID3 5.91 mm to (141.0, 134.4)
