File: kicad/nahs-HeatBrick_v1.0_r1/nahs-HeatBrick_v1.0_r1.kicad_sch (KiCad schematic)
At the start: 62 parts, among them IC1 ESP12S, IC2 ATTINY414, J2 AKL 101-02, J3 AKL 101-02, Q1 BSS138, Q3 BS170, SW1 KMR_231_G_LFS, SW2 SSSS820101, SW3 SW_DIP_x04, SW4 Taster_3301, SW5 Taster_4545, U1 MCP1700-3302, U2 LM1086_IT5,0

Commit message: v1.0 R1 ibom done
Parts:
- C1: Storage (none) -> MAG4
- FID1, FID2, FID3, J, JP1, JP10, JP11, JP12, JP13, JP2, JP3, JP4, JP5, JP6, JP7, JP9, LOGO1, LOGO2, SJ1: DNP (none) -> true
- IC1: Handsolder (none) -> true; Storage (none) -> SK1 3x5; StorageDesc (none) -> ESP12-F
- IC2: Storage (none) -> MAG4; StorageDesc (none) -> ATtiny414
- J2, J3: Handsolder (none) -> true; Storage (none) -> SB1
- LED2: value Green -> Red; Storage (none) -> MAG4; StorageDesc (none) -> LED OrangeRed
- LED3: Handsolder (none) -> true; Storage (none) -> SK1 2x5; StorageDesc (none) -> LED 5mm Red
- LED4: Handsolder (none) -> true; Storage (none) -> SK1 2x5; StorageDesc (none) -> LED 5mm Green
- LED5: Handsolder (none) -> true; Storage (none) -> SK1 2x4; StorageDesc (none) -> LED 5mm Blue
- Q1: Storage (none) -> MAG3; StorageDesc (none) -> BSS138
- Q3: Handsolder (none) -> true; Storage (none) -> SK1 1x2; StorageDesc (none) -> BS170
- R1, R2, R5, R6: Storage (none) -> MAG1
- R10, R11, R3, R4, R7, R9: Storage (none) -> MAG2
- R12, R13, R14, R15, R20, R21: Storage (none) -> MAG1; StorageDesc (none) -> 0603
- SW1: Storage (none) -> SK1 2x2; StorageDesc (none) -> KMR 231 G LFS
- SW2: Storage (none) -> SK1 2x2; StorageDesc (none) -> SSSS820101
- SW3: Handsolder (none) -> true; Storage (none) -> SK2 2x2; StorageDesc (none) -> DIP Switch 4x
- SW4, SW5: Handsolder (none) -> true; Storage (none) -> SK1 4x3; StorageDesc (none) -> Taster 4545
- U1: Storage (none) -> MAG3; StorageDesc (none) -> MCP1700
- U2: Handsolder (none) -> true; Storage (none) -> SK1 1x4; StorageDesc (none) -> LM1086 IT5,0
